File: planter_pcb.kicad_pcb (KiCad board)
At the start: 4 copper layers, 41.1 x 96.6 mm, 52 parts, among them J1 PROG_CNN, J2 Pad, Q1 MMBT3904, Q5 Si2301CDS, SW1 DSHP02TSGET, U1 STM32U031F8P6, U2 BH1750FVI, U3 TPS22917DBV, U4 SHTC3

Commit message: updated last changes
Parts:
- removed Q1: MMBT3904, Package_TO_SOT_SMD:SOT-23
- removed R2: 47K, Resistor_SMD:R_0603_1608Metric
- removed R4: 150K, Resistor_SMD:R_0603_1608Metric
- added C5: 100n, Capacitor_SMD:C_0603_1608Metric, F.Cu at (129.8, 64.5)
- added U5: 74AUP1G14, Package_TO_SOT_SMD:SOT-23-5, F.Cu at (132.6, 64.3)
- moved R5 6.37 mm to (135.4, 64.5), turned to 90 degrees
- moved TP3 0.13 mm to (137.9, 66.0)
Connections:
- BZ1 pad 1: +3V0 -> /MCU/BUZZER_IO
- R3 pad 1: +3V0 -> GND
- R5 pad 1: +3V0 -> GND
- R5 pad 2: Net-(BZ1--) -> /MCU/BUZZER_IO
Routing:
- net /MCU/BUZZER_IO: track 7.17 -> 17.4 mm
- net Net-(BZ1--): track 13.0 -> 7.58 mm
- net Net-(Q1-B): track 5.31 -> 0.00 mm
- net +3V0: track 17.7 -> 17.3 mm, vias 16 -> 14
- net GND: track 7.47 -> 7.56 mm, vias 78 -> 22
